Commit message: fix(rs_bpearl): add rate and topic params

File: robosense_description/urdf/rs_bpearl.urdf.xacro (robot description, xacro)
@@ -3,5 +3,5 @@
     <xacro:include filename="$(find robosense_description)/urdf/inertias.xacro" />
     <xacro:property name="M_PI" value="3.1415926535897931" />
-    <xacro:macro name="rs_bpearl" params="name parent_link *origin gpu:=false">
+    <xacro:macro name="rs_bpearl" params="name parent_link *origin gpu:=false rate:=10 topic:=''">
         <link name="${name}">
             <xacro:cylinder_inertial_collision_with_origin radius="0.04" length="0.08" mass="5" >
@@ -36,6 +36,6 @@
         <xacro:robosense_lidar_sensor
             name="${name}"
-            topic="${name}/points"
-            rate="10"
+            topic="${topic if topic else name+'/points'}"
+            rate="${rate}"
             lasers="32"
             samples="1800"
