Commit message: refactor(lidar model): parameterize vertical min max angles

File: robosense_description/urdf/RS-16.urdf.xacro (robot description, xacro)
@@ -2,5 +2,5 @@
 <robot xmlns:xacro="http://www.ros.org/wiki/xacro" name="RS-16">
   <xacro:property name="M_PI" value="3.1415926535897931" />
-  <xacro:macro name="RS-16" params="*origin parent:=base_link name:=robosense topic:=/robosense_points hz:=20 lasers:=16 samples:=900 collision_range:=0.4 min_range:=0.4 max_range:=150.0 noise:=0.008 min_angle:=-${M_PI} max_angle:=${M_PI} gpu:=false">
+  <xacro:macro name="RS-16" params="*origin parent:=base_link name:=robosense topic:=/robosense_points hz:=20 lasers:=16 samples:=900 collision_range:=0.4 min_range:=0.4 max_range:=150.0 noise:=0.008 min_angle:=-${M_PI} max_angle:=${M_PI} min_angle_vertical:=-${15.0*M_PI/180.0} max_angle_vertical:=-${15.0*M_PI/180.0} gpu:=false">
     <joint name="${name}_base_mount_joint" type="fixed">
       <xacro:insert_block name="origin" />
@@ -54,4 +54,6 @@
       min_angle="${min_angle}"
       max_angle="${max_angle}"
+      min_angle_vertical="${min_angle_vertical}"
+      max_angle_vertical="${max_angle_vertical}"
       gpu="${gpu}" />
   </xacro:macro>

Commit message: added ros2 humble version

File: robosense_description/urdf/RS-16.urdf.xacro (robot description, xacro)
@@ -2,5 +2,5 @@
 <robot xmlns:xacro="http://www.ros.org/wiki/xacro" name="RS-16">
   <xacro:property name="M_PI" value="3.1415926535897931" />
-  <xacro:macro name="RS-16" params="*origin parent:=base_link name:=robosense topic:=/robosense_points hz:=20 lasers:=16 samples:=900 collision_range:=0.4 min_range:=0.4 max_range:=150.0 noise:=0.008 min_angle:=-${M_PI} max_angle:=${M_PI} gpu:=false">
+  <xacro:macro name="RS-16" params="*origin parent:=base_link name:=robosense topic:=/robosense_points hz:=20 lasers:=16 samples:=360 collision_range:=0.4 min_range:=0.4 max_range:=150.0 noise:=0.008 min_angle:=-${M_PI} max_angle:=${M_PI} gpu:=false">
     <joint name="${name}_base_mount_joint" type="fixed">
       <xacro:insert_block name="origin" />
@@ -74,10 +74,14 @@
             </noise>
           </ray>
-          <plugin name="gazebo_ros_laser_controller" filename="libgazebo_ros_robosense_gpu_laser.so">
-            <topicName>${topic}</topicName>
+          <plugin name="gazebo_ros_laser_controller" filename="libgazebo_ros_robosense_laser.so">
+            <ros>
+              <namespace>/${name}</namespace>
+              <remapping>~/out:=${topic}</remapping>
+            </ros>
+            <tf_prefix>${tf_prefix}</tf_prefix>
             <frameName>${name}</frameName>
             <min_range>${min_range}</min_range>
             <max_range>${max_range}</max_range>
-            <gaussianNoise>${noise}</gaussianNoise>
+            <gaussian_noise>${noise}</gaussian_noise>
           </plugin>
         </sensor>
@@ -86,4 +90,5 @@
         <sensor type="ray" name="${name}-RS16">
           <pose>0 0 0 0 0 0</pose>
+          <always_on>true</always_on>
           <visualize>false</visualize>
           <update_rate>${hz}</update_rate>
@@ -115,9 +120,12 @@
           </ray>
           <plugin name="gazebo_ros_laser_controller" filename="libgazebo_ros_robosense_laser.so">
-            <topicName>${topic}</topicName>
+            <ros>
+              <namespace>/${name}</namespace>
+              <remapping>~/out:=${topic}</remapping>
+            </ros>
             <frameName>${name}</frameName>
             <min_range>${min_range}</min_range>
             <max_range>${max_range}</max_range>
-            <gaussianNoise>${noise}</gaussianNoise>
+            <gaussian_noise>${noise}</gaussian_noise>
           </plugin>
         </sensor>

File: robosense_description/urdf/example.urdf.xacro (robot description, xacro)
@@ -31,6 +31,6 @@
   </link>
   <xacro:include filename="$(find robosense_description)/urdf/RS-16.urdf.xacro"/>
-  <RS-16 parent="base_link" name="robosense" topic="/rs_points" hz="20" samples="900" gpu="${gpu}">
+  <xacro:RS-16 parent="base_link" name="robosense" topic="/rs_points" hz="20" samples="360" gpu="${gpu}">
     <origin xyz="0 0 0.4" rpy="0 0 0" />
-  </RS-16>
+  </xacro:RS-16>
 </robot>
